Commit message: Include Dimensions

File: rover_description/urdf/rover.xacro (robot description, xacro)
@@ -12,5 +12,5 @@
         <visual>
             <geometry>
-                <box size="0.6 0.1 0.2"/>
+                <box size="0.28 0.14 0.082"/>
             </geometry>
             <origin rpy="0 0 0" xyz="0 0 0"/>
@@ -19,5 +19,5 @@
         <collision>
             <geometry>
-                <box size="0.6 0.1 0.2"/>
+                <box size="0.28 0.14 0.082"/>
             </geometry>
             <origin rpy="0 0 0" xyz="0 0 0"/>
@@ -31,5 +31,5 @@
         <parent link="base_link"/>
         <child link="chassis"/>
-        <origin xyz="0 0 0"/>
+        <origin xyz="0 0 0.0615"/>
     </joint>
     <!-- Define the wheels -->
@@ -38,14 +38,14 @@
             <visual>
                 <geometry>
-                    <cylinder length="0.6" radius="0.2"/>
+                    <cylinder length="0.035" radius="0.035"/>
                 </geometry>
-                <origin rpy="0 0 0" xyz="0 0 0"/>
+                <origin rpy="1.57 0 0" xyz="0 0 0"/>
                 <material name="black"/>
             </visual>
             <collision>
                 <geometry>
-                    <cylinder length="0.6" radius="0.2"/>
+                    <cylinder length="0.035" radius="0.035"/>
                 </geometry>
-                <origin rpy="0 0 0" xyz="0 0 0"/>
+                <origin rpy="1.57 0 0" xyz="0 0 0"/>
             </collision>
             <inertial>
@@ -63,9 +63,9 @@
     </xacro:macro>
     <!-- Create 6 wheels -->
-    <xacro:wheel prefix="wheel1" xyz="0.2 0.01 0"/>
-    <xacro:wheel prefix="wheel2" xyz="0.2 0.01 0"/>
-    <xacro:wheel prefix="wheel3" xyz="0.2 0.01 0"/>
-    <xacro:wheel prefix="wheel4" xyz="0.2 0.01 0"/>
-    <xacro:wheel prefix="wheel5" xyz="0.2 0.01 0"/>
-    <xacro:wheel prefix="wheel6" xyz="0.2 0.01 0"/>
+    <xacro:wheel prefix="wheel1" xyz="0.105 0.0925 -0.031"/>
+    <xacro:wheel prefix="wheel2" xyz="0.105 -0.0925 -0.031"/>
+    <xacro:wheel prefix="wheel3" xyz="0.0 0.0925 -0.031"/>
+    <xacro:wheel prefix="wheel4" xyz="0.0 -0.0925 -0.031"/>
+    <xacro:wheel prefix="wheel5" xyz="-0.105 0.0925 -0.031"/>
+    <xacro:wheel prefix="wheel6" xyz="-0.105 -0.0925 -0.031"/>
 </robot>

Commit message: Add realsense

File: rover_description/urdf/rover.xacro (robot description, xacro)
@@ -33,4 +33,8 @@
         <origin xyz="0 0 0.0615"/>
     </joint>
+    <xacro:include filename="$(find realsense2_description)/urdf/_d435.urdf.xacro" />
+    <xacro:sensor_d435 name="camera" parent="chassis">
+        <origin xyz="0.12 0.0 0.071" rpy="0 0 0"/>
+    </xacro:sensor_d435>
     <!-- Define the wheels -->
     <xacro:macro name="wheel" params="prefix xyz">
